File: hardware/stm32_sniffer/stm32_sniffer.kicad_sch (KiCad schematic)
At the start: 3 parts, among them J1 APPLE_SDISKII, J2 APPLE_SDISKII

Commit message: hardware pcb
Parts:
- added D1, D2: LED, LED_THT:LED_D5.0mm, symbol Device:LED
- added J4: Conn_02x05_Odd_Even, Connector_IDC:IDC-Header_2x05_P2.54mm_Vertical, symbol Connector_Generic:Conn_02x05_Odd_Even
- added J5: STLINK, Connector_PinHeader_2.54mm:PinHeader_1x04_P2.54mm_Vertical, symbol Connector:Conn_01x04_Pin
- added J6: PWR, Connector_PinHeader_2.54mm:PinHeader_1x02_P2.54mm_Vertical, symbol Connector:Conn_01x02_Pin
- added J7: UART, Connector_PinHeader_2.54mm:PinHeader_1x03_P2.54mm_Vertical, symbol Connector:Conn_01x03_Pin
- added J8: APPLE_SDISKII, Connector_PinHeader_2.54mm:PinHeader_2x10_P2.54mm_Vertical, symbol Connector_Generic:Conn_02x10_Odd_Even
- added JP1: SPST, Jumper:SolderJumper-2_P1.3mm_Open_RoundedPad1.0x1.5mm, symbol Jumper:SolderJumper_2_Open
- added R1, R2: 68R, Resistor_THT:R_Axial_DIN0207_L6.3mm_D2.5mm_P7.62mm_Horizontal, symbol Device:R
- added SW_BTN_ENTR1: SW_Push, Button_Switch_THT:SW_PUSH_6mm, symbol Switch:SW_Push
- added U2: MicroSD_SPI_CD, sdisk_stm32:GCT-MEM2055-00-190-01-A, symbol microsd_spi_cd:MicroSD_SPI_CD
Connections:
- net SPI_NSS: now reaches μC1.1 (B12)
- net SPI_NSS: now also U2.2 (D3)
- net DEBUG1: now reaches μC1.10 (A15)
- net DEBUG1: now also J4.1 (Pin_1), J8.1 (Pin_1)
- net TIM2CH2: now reaches μC1.11 (B3)
- net TIM2CH2: now also J8.14 (Pin_14)
- net DEBUG2: now reaches μC1.12 (B4)
- net DEBUG2: now also J4.2 (Pin_2), J8.2 (Pin_2)
- net DEVICE_ENABLE: now reaches μC1.13 (B5)
- net DEVICE_ENABLE: now also J1.14 (Pin_14), J2.14 (Pin_14), J4.3 (Pin_3), J8.11 (Pin_11)
- net LED1: now reaches μC1.14 (B6)
- net LED1: now also R1.2
- net LED2: now reaches μC1.15 (B7)
- net LED2: now also R2.2
- net SD_EJECT: now reaches μC1.16 (B8)
- net SD_EJECT: now also U2.8 (D1)
- net WR_REQ: now reaches μC1.17 (B9)
- net WR_REQ: now also J1.10 (Pin_10), J2.10 (Pin_10), J4.7 (Pin_7), J8.9 (Pin_9)
- net PWR_IN: now reaches μC1.18 (5Vi)
- net PWR_IN: now also J6.2 (Pin_2), JP1.1 (A)
- net GND: now reaches μC1.19 (GNDi)
- net GND: now also J1.1 (Pin_1), J1.3 (Pin_3), J1.5 (Pin_5), J2.1 (Pin_1), J2.3 (Pin_3), J2.5 (Pin_5), μC1.39 (GNDii), μC1.44 (GND), D1.1 (K), D2.1 (K), J4.10 (Pin_10), J4.9 (Pin_9), J5.4 (Pin_4), J7.3 (Pin_3), J8.19 (Pin_19), J8.20 (Pin_20), U2.10 (GND), U2.6 (GND)
- net SPI_SCK: now reaches μC1.2 (B13)
- net SPI_SCK: now also U2.5 (SCLK)
- net 3.3V: now reaches μC1.20 (3.3i)
- net 3.3V: now also SW_BTN_ENTR1.1
- net PHASE0: now reaches μC1.26 (A0)
- net PHASE0: now also J1.2 (Pin_2), J2.2 (Pin_2), J8.3 (Pin_3)
- net PHASE1: now reaches μC1.27 (A1)
- net PHASE1: now also J1.4 (Pin_4), J2.4 (Pin_4), J8.4 (Pin_4)
- net PHASE2: now reaches μC1.28 (A2)
- net PHASE2: now also J1.6 (Pin_6), J2.6 (Pin_6), J8.5 (Pin_5)
- net PHASE3: now reaches μC1.29 (A3)
- net PHASE3: now also J1.8 (Pin_8), J2.8 (Pin_8), J8.6 (Pin_6)
- net SPI_MISO: now reaches μC1.3 (B14)
- net SPI_MISO: now also U2.7 (DO)
- net TIM2ETR: now reaches μC1.31 (A5)
- net TIM2ETR: now also J1.18 (Pin_18), J2.18 (Pin_18), μC1.33 (A7), J4.6 (Pin_6), J8.8 (Pin_8)
- net RD_DATA: now reaches μC1.32 (A6)
- net RD_DATA: now also J1.16 (Pin_16), J2.16 (Pin_16), μC1.9 (A12), J4.5 (Pin_5), J8.7 (Pin_7)
- net WR_PROTECT: now reaches μC1.37 (B10)
- net WR_PROTECT: now also J1.20 (Pin_20), J2.20 (Pin_20), J4.8 (Pin_8), J8.10 (Pin_10)
- net +3.3V: now reaches μC1.38 (3.3ii)
- net +3.3V: now also μC1.41 (3.3V), J5.1 (Pin_1), U2.4 (VDD)
- net SPI_MOSI: now reaches μC1.4 (B15)
- net SPI_MOSI: now also U2.3 (CMD)
- net SDIO: now reaches μC1.42 (SDIO)
- net SDIO: now also J5.2 (Pin_2)
- net SCK: now reaches μC1.43 (SCK)
- net SCK: now also J5.3 (Pin_3)
- net TIM1CH1: now reaches μC1.5 (A8)
- net TIM1CH1: now also J8.13 (Pin_13)
- net UART_TX: now reaches μC1.6 (A9)
- net UART_TX: now also J7.1 (Pin_1)
- net UART_RX: now reaches μC1.7 (A10)
- net UART_RX: now also J7.2 (Pin_2)
- net BTN1: now reaches μC1.8 (A11)
- net BTN1: now also SW_BTN_ENTR1.2
- net VCC: now reaches J1.11 (Pin_11)
- net VCC: now also J2.11 (Pin_11), J6.1 (Pin_1), JP1.2 (B)
- net SELECT: now reaches J1.12 (Pin_12)
- net SELECT: now also J2.12 (Pin_12), J4.4 (Pin_4), J8.12 (Pin_12)
- net P12: now reaches J1.13 (Pin_13)
- net P12: now also J1.15 (Pin_15), J1.17 (Pin_17), J1.19 (Pin_19), J2.13 (Pin_13), J2.15 (Pin_15), J2.17 (Pin_17), J2.19 (Pin_19)
- net DISK3.5: now reaches J1.7 (Pin_7)
- net DISK3.5: now also J2.7 (Pin_7), J8.15 (Pin_15)
- net M12: now reaches J1.9 (Pin_9)
- net M12: now also J2.9 (Pin_9)
- new net: D1.2 (A), R1.1
- new net: D2.2 (A), R2.1
- no-connect marks 0 -> 11
Other:
- moved on the sheet: J2
